Commit message: commit robotmovbile+camera

File: ros2_iiwa/iiwa_description/urdf/iiwa.urdf.xacro (robot description, xacro)
@@ -240,5 +240,5 @@
         </geometry>
         <material>
-          <color rgba="0.0 1.0 0.0 1.0"/> <!-- Verde per distinguere la camera -->
+          <color rgba="0.0 0.0 0.0 1.0"/> <!-- Verde per distinguere la camera -->
         </material>
       </visual>
@@ -251,5 +251,5 @@
     <!-- Joint per collegare la camera -->
     <joint name="${prefix}camera_joint" type="fixed">
-      <origin xyz="0 0 0.11" rpy="0 -1.57 0"/> <!-- Posizionata sull'end-effector -->
+      <origin xyz="0 0 0" rpy="0 -1.57 0"/> <!-- Posizionata sull'end-effector -->
       <parent link="${prefix}tool0"/>
       <child link="${prefix}camera_link"/>

Commit message: aruco marker detector

File: ros2_iiwa/iiwa_description/urdf/iiwa.urdf.xacro (robot description, xacro)
@@ -225,5 +225,5 @@
       <axis xyz="0 0 0"/>
   </joint>
-  <!--<xacro:if value="${use_vision}">-->
+  <xacro:if value="${use_vision}">
     <xacro:include filename="$(find iiwa_description)/urdf/iiwa_camera.xacro"/>
     <xacro:iiwa_camera reference="camera_link"/>
@@ -251,10 +251,10 @@
     <!-- Joint per collegare la camera -->
     <joint name="${prefix}camera_joint" type="fixed">
-      <origin xyz="0 0 0" rpy="0 -1.57 0"/> <!-- Posizionata sull'end-effector -->
+      <origin xyz="0 0 0" rpy="0 0 0"/> <!-- Posizionata sull'end-effector -->
       <parent link="${prefix}tool0"/>
       <child link="${prefix}camera_link"/>
       <axis xyz="0 0 0"/>
     </joint>
-  <!--</xacro:if>-->
+  </xacro:if>
   </xacro:macro>
 </robot>

File: ros2_iiwa/iiwa_description/urdf/iiwa_camera.xacro (robot description, xacro)
@@ -9,4 +9,5 @@
     <gazebo reference="${reference}">
       <sensor name="camera" type="camera">
+        <pose>0 0 0 0 -1.57 0</pose>
         <camera>
           <horizontal_fov>1.047</horizontal_fov>
